Commit message: Updated name to match gummi package name convention

File: xacro/gummi_description_head.urdf.xacro (robot description, xacro)
@@ -23,5 +23,5 @@
         <geometry>
           <mesh
-            filename="package://two_dof_head/meshes/head_yaw.stl" />
+            filename="package://gummi_head_$(env ROS_GUMMI_HEAD)/meshes/head_yaw.stl" />
         </geometry>
         <material
@@ -37,5 +37,5 @@
         <geometry>
           <mesh
-            filename="package://two_dof_head/meshes/head_yaw_CH.stl" />
+            filename="package://gummi_head_$(env ROS_GUMMI_HEAD)/meshes/head_yaw_CH.stl" />
         </geometry>
       </collision>
@@ -79,5 +79,5 @@
           <geometry>
             <mesh
-              filename="package://two_dof_head/meshes/head_pitch.stl" />
+              filename="package://gummi_head_$(env ROS_GUMMI_HEAD)/meshes/head_pitch.stl" />
           </geometry>
           <material
@@ -93,5 +93,5 @@
           <geometry>
             <mesh
-              filename="package://two_dof_head/meshes/head_pitch_CH.stl" />
+              filename="package://gummi_head_$(env ROS_GUMMI_HEAD)/meshes/head_pitch_CH.stl" />
           </geometry>
         </collision>

File: xacro/gummi_head.srdf.xacro (robot description, xacro)
@@ -1,9 +1,9 @@
 <?xml version="1.0" ?>
 <robot name="gummi" xmlns:xacro="http://www.ros.org/wiki/xacro">
-<xacro:macro name="head">
+<xacro:macro name="two_dof_head">
     <joint name="head_yaw" />
     <joint name="head_pitch" />
 </xacro:macro>
-<xacro:macro name="group_state_head">
+<xacro:macro name="group_state_two_dof_head">
   <joint name="head_yaw" value="0" />
   <joint name="head_pitch" value="0" />

Commit message: Required Functionality for Moving Head
Added the functionality required to get the head moving in MoveIt!

File: xacro/gummi_description_head.urdf.xacro (robot description, xacro)
@@ -52,5 +52,5 @@
         link="head_yaw" />
       <axis
-        xyz="0 0 1" />
+        xyz="0 0 -1" />
       <limit
         effort="0"

File: xacro/gummi_head.srdf.xacro (robot description, xacro)
@@ -1,11 +1,15 @@
 <?xml version="1.0" ?>
 <robot name="gummi" xmlns:xacro="http://www.ros.org/wiki/xacro">
-<xacro:macro name="two_dof_head">
+<xacro:macro name="group_head_twodof">
     <joint name="head_yaw" />
     <joint name="head_pitch" />
 </xacro:macro>
-<xacro:macro name="group_state_two_dof_head">
+<xacro:macro name="group_state_head_twodof">
   <joint name="head_yaw" value="0" />
   <joint name="head_pitch" value="0" />
+</xacro:macro>
+<xacro:macro name="virtual_joints_base">
+  <!--VIRTUAL JOINT: Purpose: this element defines a virtual joint between a robot link and an external frame of reference (considered fixed with respect to the robot)-->
+  <virtual_joint name="virtual_joint" type="fixed" parent_frame="map" child_link="base_link" />
 </xacro:macro>
 <xacro:macro name="disable_collisions_head">

Commit message: Added the camera to the serial chain

File: xacro/gummi_description_head.urdf.xacro (robot description, xacro)
@@ -113,3 +113,56 @@
           velocity="1" />
       </joint>
-  </robot>
+      <link
+        name="camera">
+        <inertial>
+          <origin
+           xyz="0.0484512742480244 0.0139768664666073 0.000956995637939325"
+           rpy="0 0 0" />
+        <mass
+           value="0.0644774651698934" />
+        <inertia
+        ixx="8.67406414845019E-06"
+        ixy="-1.3193756197629E-05"
+        ixz="-3.41916035169704E-06"
+        iyy="4.217442276821E-05"
+        iyz="-4.04257224014858E-07"
+        izz="4.91399139463636E-05" />
+        </inertial>
+        <visual>
+          <origin
+          xyz="0 0 0"
+          rpy="0 0 0" />
+        <geometry>
+          <mesh
+           filename="package://gummi_head_$(env ROS_GUMMI_HEAD)/meshes/realsense_CH.stl" />
+        </geometry>
+        <material
+          name="">
+          <color
+            rgba="0.792156862745098 0.819607843137255 0.933333333333333 1" />
+        </material>
+        </visual>
+        <collision>
+          <origin
+            xyz="0 0 0"
+            rpy="0 0 0" />
+        <geometry>
+         <mesh
+            filename="package://gummi_head_$(env ROS_GUMMI_HEAD)/meshes/realsense_CH.stl" />
+        </geometry>
+        </collision>
+    </link>
+   <joint
+      name="camera"
+      type="fixed">
+      <origin
+        xyz="0.05 0.022 0"
+        rpy="0 1.57079632679 0" />
+      <parent
+        link="head_pitch" />
+      <child
+        link="camera" />
+      <axis
+        xyz="0 0 0" />
+    </joint>
+</robot>

File: xacro/gummi_head.srdf.xacro (robot description, xacro)
@@ -4,4 +4,5 @@
     <joint name="head_yaw" />
     <joint name="head_pitch" />
+    <joint name="camera" />
 </xacro:macro>
 <xacro:macro name="group_state_head_twodof">
@@ -17,4 +18,7 @@
   <disable_collisions link1="head_yaw" link2="head_pitch" reason="Adjacent" />
   <disable_collisions link1="base_link" link2="head_pitch" reason="Never" />
+  <disable_collisions link1="base_link" link2="camera" reason="Never"/>
+  <disable_collisions link1="head_pitch" link2="camera" reason="Adjacent" />
+  <disable_collisions link1="head_yaw" link2="camera" reason="Never" />
 </xacro:macro>
 </robot>
